File: pcb/wifi extension inspired/PCB_WiFiModule to Xbee rev0.2.brd (EAGLE design)
At the start: 40.5 x 32.5 mm, 20 parts, among them J1 FA12-1W, U1 XBP9B-DMUT-002

Commit message: cleaned up routing, rerouted some SJ to go to different GPIO on the Xbee module.
Connections:
- net N$10: now also SJ2.2; no longer SJ3.2
- net N$11: now also SJ3.2; no longer SJ2.2
Routing:
- net N$10: track 10.2 -> 4.39 mm
- net RE0: track 20.7 -> 19.2 mm, vias 0 -> 1
- net N$11: track 17.5 -> 18.6 mm, vias 0 -> 1
Changed lines of the file:
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@@
 <via x="4.7625" y="28.575" extent="1-16" drill="0.3"/>
 <via x="4.7625" y="31.115" extent="1-16" drill="0.3"/>
+<via x="19.3675" y="1.5875" extent="1-16" drill="0.3"/>
+<via x="6.0325" y="26.67" extent="1-16" drill="0.3"/>
+<via x="29.21" y="19.05" extent="1-16" drill="0.3"/>
+<via x="38.4175" y="6.985" extent="1-16" drill="0.3"/>
+<via x="38.4175" y="1.905" extent="1-16" drill="0.3"/>
+<via x="28.2575" y="1.5875" extent="1-16" drill="0.3"/>
+<via x="24.765" y="11.7475" extent="1-16" drill="0.3"/>
+<via x="29.21" y="11.7475" extent="1-16" drill="0.3"/>
+<via x="19.685" y="11.7475" extent="1-16" drill="0.3"/>
+<via x="37.1475" y="12.3825" extent="1-16" drill="0.3"/>
+<via x="37.1475" y="19.3675" extent="1-16" drill="0.3"/>
+<via x="37.1475" y="15.875" extent="1-16" drill="0.3"/>
+<via x="21.2725" y="15.5575" extent="1-16" drill="0.3"/>
+<via x="24.765" y="15.5575" extent="1-16" drill="0.3"/>
+<via x="29.21" y="15.5575" extent="1-16" drill="0.3"/>
+<via x="17.78" y="23.1775" extent="1-16" drill="0.3"/>
+<via x="17.78" y="25.0825" extent="1-16" drill="0.3"/>
+<via x="19.05" y="24.13" extent="1-16" drill="0.3"/>
+<via x="20.32" y="23.1775" extent="1-16" drill="0.3"/>
+<via x="20.32" y="25.0825" extent="1-16" drill="0.3"/>
+<via x="21.59" y="24.13" extent="1-16" drill="0.3"/>
 </signal>
 <signal name="VBAT">
@@
 <contactref element="J1" pad="11"/>
 <contactref element="U1" pad="13"/>
-<wire x1="2.51" y1="5" x2="4.495" y2="6.985" width="0.2032" layer="1"/>
-<wire x1="11.1125" y1="6.985" x2="12.065" y2="6.0325" width="0.2032" layer="1"/>
-<wire x1="12.065" y1="6.0325" x2="12.065" y2="4.1275" width="0.2032" layer="1"/>
-<wire x1="12.065" y1="4.1275" x2="12.7" y2="3.4925" width="0.2032" layer="1"/>
-<wire x1="4.495" y1="6.985" x2="11.1125" y2="6.985" width="0.2032" layer="1"/>
-<wire x1="18.605" y1="4.3175" x2="18.605" y2="5.23" width="0.2032" layer="1"/>
-<wire x1="12.7" y1="3.4925" x2="17.78" y2="3.4925" width="0.2032" layer="1"/>
-<wire x1="17.78" y1="3.4925" x2="18.605" y2="4.3175" width="0.2032" layer="1"/>
+<wire x1="2.51" y1="5" x2="9.605" y2="5" width="0.2032" layer="16"/>
+<wire x1="12.3825" y1="2.2225" x2="16.8275" y2="2.2225" width="0.2032" layer="16"/>
+<via x="16.8275" y="2.2225" extent="1-16" drill="0.3"/>
+<wire x1="16.8275" y1="2.2225" x2="18.605" y2="4" width="0.2032" layer="1"/>
+<wire x1="18.605" y1="4" x2="18.605" y2="5.23" width="0.2032" layer="1"/>
+<wire x1="9.605" y1="5" x2="12.3825" y2="2.2225" width="0.2032" layer="16"/>
 </signal>
 <signal name="RF1">
@@
 <contactref element="R4" pad="2"/>
 <contactref element="U1" pad="15"/>
-<wire x1="22.605" y1="5.23" x2="22.605" y2="5.97" width="0.2032" layer="1"/>
-<wire x1="21.59" y1="6.985" x2="18.7325" y2="6.985" width="0.2032" layer="1"/>
-<wire x1="18.7325" y1="6.985" x2="17.78" y2="7.9375" width="0.2032" layer="1"/>
-<wire x1="17.78" y1="7.9375" x2="17.78" y2="17.4625" width="0.2032" layer="1"/>
-<wire x1="17.78" y1="17.4625" x2="15.5575" y2="19.685" width="0.2032" layer="1"/>
-<wire x1="15.5575" y1="19.685" x2="10.16" y2="19.685" width="0.2032" layer="1"/>
-<wire x1="10.16" y1="19.685" x2="8.5725" y2="21.2725" width="0.2032" layer="1"/>
-<wire x1="8.5725" y1="21.2725" x2="8.5725" y2="23.0251" width="0.2032" layer="1"/>
-<wire x1="22.605" y1="5.97" x2="21.59" y2="6.985" width="0.2032" layer="1"/>
+<wire x1="22.605" y1="5.23" x2="22.605" y2="16.13" width="0.2032" layer="1"/>
+<wire x1="22.605" y1="16.13" x2="19.685" y2="19.05" width="0.2032" layer="1"/>
+<wire x1="19.685" y1="19.05" x2="18.0975" y2="19.05" width="0.2032" layer="1"/>
+<wire x1="18.0975" y1="19.05" x2="16.51" y2="20.6375" width="0.2032" layer="1"/>
+<wire x1="16.51" y1="20.6375" x2="9.525" y2="20.6375" width="0.2032" layer="1"/>
+<wire x1="9.525" y1="20.6375" x2="8.5725" y2="21.59" width="0.2032" layer="1"/>
+<wire x1="8.5725" y1="21.59" x2="8.5725" y2="23.0251" width="0.2032" layer="1"/>
 </signal>
 <signal name="N$9">
 <contactref element="U1" pad="12"/>
 <contactref element="SJ4" pad="2"/>
-<wire x1="16.605" y1="5.23" x2="16.605" y2="11.335" width="0.2032" layer="1"/>
-<wire x1="16.605" y1="11.335" x2="12.065" y2="15.875" width="0.2032" layer="1"/>
-<wire x1="12.065" y1="15.875" x2="10.287" y2="15.875" width="0.2032" layer="1"/>
+<wire x1="16.605" y1="5.23" x2="16.605" y2="11.6525" width="0.2032" layer="1"/>
+<wire x1="16.605" y1="11.6525" x2="12.3825" y2="15.875" width="0.2032" layer="1"/>
+<wire x1="12.3825" y1="15.875" x2="10.287" y2="15.875" width="0.2032" layer="1"/>
 </signal>
 <signal name="N$10">
 <contactref element="U1" pad="11"/>
+<contactref element="SJ2" pad="2"/>
+<wire x1="10.287" y1="5.3975" x2="13.0175" y2="5.3975" width="0.2032" layer="1"/>
+<wire x1="13.0175" y1="5.3975" x2="13.185" y2="5.23" width="0.2032" layer="1"/>
+<wire x1="13.185" y1="5.23" x2="13.485" y2="5.23" width="0.2032" layer="1"/>
+<wire x1="13.485" y1="5.23" x2="14.605" y2="5.23" width="0.2032" layer="1"/>
+</signal>
+<signal name="N$11">
+<contactref element="U1" pad="16"/>
 <contactref element="SJ3" pad="2"/>
-<wire x1="14.605" y1="5.23" x2="14.605" y2="10.16" width="0.2032" layer="1"/>
-<wire x1="14.605" y1="10.16" x2="12.3825" y2="12.3825" width="0.2032" layer="1"/>
-<wire x1="12.3825" y1="12.3825" x2="10.287" y2="12.3825" width="0.2032" layer="1"/>
-</signal>
-<signal name="N$11">
-<contactref element="SJ2" pad="2"/>
-<contactref element="U1" pad="16"/>
-<wire x1="10.287" y1="5.3975" x2="10.287" y2="4.0005" width="0.2032" layer="1"/>
-<wire x1="24.605" y1="4.285" x2="24.605" y2="5.23" width="0.2032" layer="1"/>
-<wire x1="10.287" y1="4.0005" x2="11.1506" y2="3.1369" width="0.2032" layer="1"/>
-<wire x1="11.1506" y1="3.1369" x2="23.4569" y2="3.1369" width="0.2032" layer="1"/>
-<wire x1="23.4569" y1="3.1369" x2="24.605" y2="4.285" width="0.2032" layer="1"/>
+<wire x1="10.287" y1="12.3825" x2="12.065" y2="12.3825" width="0.2032" layer="1"/>
+<wire x1="12.065" y1="12.3825" x2="15.24" y2="9.2075" width="0.2032" layer="1"/>
+<via x="15.24" y="9.2075" extent="1-16" drill="0.3"/>
+<wire x1="15.24" y1="9.2075" x2="22.86" y2="9.2075" width="0.2032" layer="16"/>
+<wire x1="24.605" y1="7.4625" x2="24.605" y2="5.23" width="0.2032" layer="16"/>
+<wire x1="22.86" y1="9.2075" x2="24.605" y2="7.4625" width="0.2032" layer="16"/>
 </signal>
 <signal name="N$12">
@@
 <wire x1="27.7749" y1="6.8326" x2="28.605" y2="6.0025" width="0.2032" layer="1"/>
 </signal>
-<signal name="DGND1">
-<via x="37.1475" y="12.3825" extent="1-16" drill="0.3"/>
-<via x="37.1475" y="19.3675" extent="1-16" drill="0.3"/>
-<via x="37.1475" y="15.875" extent="1-16" drill="0.3"/>
-</signal>
-<signal name="DGND2">
-<via x="38.4175" y="6.985" extent="1-16" drill="0.3"/>
-<via x="38.4175" y="1.905" extent="1-16" drill="0.3"/>
-<via x="28.2575" y="1.5875" extent="1-16" drill="0.3"/>
-</signal>
-<signal name="DGND3">
-<via x="19.3675" y="1.5875" extent="1-16" drill="0.3"/>
-<via x="6.0325" y="26.67" extent="1-16" drill="0.3"/>
-<via x="29.21" y="19.05" extent="1-16" drill="0.3"/>
-</signal>
-<signal name="DGND4">
-<via x="21.2725" y="15.5575" extent="1-16" drill="0.3"/>
-<via x="24.765" y="15.5575" extent="1-16" drill="0.3"/>
-<via x="29.21" y="15.5575" extent="1-16" drill="0.3"/>
-</signal>
-<signal name="DGND5">
-<via x="24.765" y="11.7475" extent="1-16" drill="0.3"/>
-<via x="29.21" y="11.7475" extent="1-16" drill="0.3"/>
-<via x="19.685" y="11.7475" extent="1-16" drill="0.3"/>
-</signal>
-<signal name="DGND6">
-<via x="17.78" y="23.1775" extent="1-16" drill="0.3"/>
-<via x="17.78" y="25.0825" extent="1-16" drill="0.3"/>
-<via x="19.05" y="24.13" extent="1-16" drill="0.3"/>
-</signal>
-<signal name="DGND7">
-<via x="20.32" y="23.1775" extent="1-16" drill="0.3"/>
-<via x="20.32" y="25.0825" extent="1-16" drill="0.3"/>
-<via x="21.59" y="24.13" extent="1-16" drill="0.3"/>
-</signal>
 </signals>

Commit message: rev1.0 ready for review.
Parts:
- removed LED1: (no value), adafruit:CHIP-LED0603
- added STAT: (no value), adafruit:CHIP-LED0603
- moved R4 5.71 mm to (14.3, 23.8)
- moved R2 1.91 mm to (10.5, 23.8)
- moved R1 1.90 mm to (12.4, 23.8)
- moved R3 1.90 mm to (8.57, 23.8)
- moved R5 1.59 mm to (23.8, 25.1), turned to 180 degrees
- renumbered LED2 to RX, LED3 to TX, LED4 to POWER
Connections:
- net DGND: now also STAT.C; no longer TX.C
- net N$1: now also STAT.A; no longer POWER.A
- net N$2: now also RX.A; no longer LED1.A
- net N$3: now also TX.A; no longer RX.A
- net N$8: now also POWER.A; no longer TX.A
- net U6RX: now also RX.C; no longer LED1.C
- net U6TX: now also TX.C; no longer RX.C
Routing:
- net DIO5: track 28.6 -> 21.2 mm
- net U6TX: track 69.6 -> 64.9 mm
- net U6RX: track 53.6 -> 49.6 mm, vias 1 -> 3
- net +3.3V: track 66.0 -> 68.4 mm
- net N$2: track 6.44 -> 4.94 mm
- net N$1: track 5.47 -> 6.04 mm
Other:
- outline, holes or cut-outs redrawn
