File: pcb/wifi extension inspired/PCB_WiFiModule to Xbee rev1.0.brd (EAGLE design)
At the start: 40.5 x 32.5 mm, 20 parts, among them J1 FA12-1W, U1 XBP9B-DMUT-002

Commit message: rev1.0 ready for review.
Parts:
- removed LED1: (no value), adafruit:CHIP-LED0603
- added STAT: (no value), adafruit:CHIP-LED0603
- moved R4 5.71 mm to (14.3, 23.8)
- moved R2 1.91 mm to (10.5, 23.8)
- moved R1 1.90 mm to (12.4, 23.8)
- moved R3 1.90 mm to (8.57, 23.8)
- moved R5 1.59 mm to (23.8, 25.1), turned to 180 degrees
- renumbered LED2 to RX, LED3 to TX, LED4 to POWER
Connections:
- net DGND: now also STAT.C; no longer TX.C
- net N$1: now also STAT.A; no longer POWER.A
- net N$2: now also RX.A; no longer LED1.A
- net N$3: now also TX.A; no longer RX.A
- net N$8: now also POWER.A; no longer TX.A
- net U6RX: now also RX.C; no longer LED1.C
- net U6TX: now also TX.C; no longer RX.C
Routing:
- net DIO5: track 28.6 -> 21.2 mm
- net U6TX: track 69.6 -> 64.9 mm
- net U6RX: track 53.6 -> 50.4 mm, vias 1 -> 3
- net +3.3V: track 66.0 -> 69.1 mm
- net N$2: track 6.44 -> 5.21 mm
- net N$1: track 5.47 -> 6.38 mm
